File: hackducky.kicad_pcb (KiCad board)
At the start: 2 copper layers, 20 x 60 mm, 41 parts, among them J1 USB_A, J2 Conn_01x06_Pin, J3 Micro_SD_Card, J4 Conn_01x06_Pin, P2 USB_C_Plug, SW3 bootsel, SW4 SW_Push, U1 W25Q16JVSS, U2 AP2112K-3.3, U4 RP2040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

Commit message: second
Parts:
- moved Y1 37.2 mm to (87.8, 85.1)
Changed lines of the file:
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@@
 	(footprint "Crystal:Crystal_SMD_1210-4Pin_1.2x1.0mm"
 		(layer "F.Cu")
-		(at 124.165 77.09)
+		(at 87.835 85.09)
 		(descr "SMD Crystal SERIES SMD1210/4 https://ecsxtal.com/store/pdf/ECX-1048.pdf, 1.2x1.0mm^2 package")
 		(tags "SMT")

Commit message: pcb layout
Parts:
- added BZ1: Buzzer, Buzzer_Beeper:Buzzer_CUI_CPT-9019S-SMT, F.Cu at (171.7, 69.5)
- added D2: MBR1020VL, Diode_SMD:D_SOD-123F, F.Cu at (153.0, 76.4)
- added D3: MBR1020VL, Diode_SMD:D_SOD-123F, F.Cu at (153.0, 79.8)
- added D4: WS2812B, LED_SMD:LED_WS2812B-2020_PLCC4_2.0x2.0mm, F.Cu at (179.6, 69.5)
- added D5: WS2812B, LED_SMD:LED_WS2812B-2020_PLCC4_2.0x2.0mm, F.Cu at (179.6, 73.1)
- added D6: WS2812B, LED_SMD:LED_WS2812B-2020_PLCC4_2.0x2.0mm, F.Cu at (179.6, 76.7)
- added D7: WS2812B, LED_SMD:LED_WS2812B-2020_PLCC4_2.0x2.0mm, F.Cu at (179.6, 80.2)
- added J5: Conn_01x03_Pin, Connector_PinSocket_2.54mm:PinSocket_1x03_P2.54mm_Vertical, F.Cu at (179.0, 53.1)
- added SW2: SW_DIP_x04, Button_Switch_THT:SW_DIP_SPSTx04_Slide_6.7x11.72mm_W7.62mm_P2.54mm_LowProfile, F.Cu at (167.5, 53.7)
- added U3: USBLC6-2P6, Package_TO_SOT_SMD:SOT-666, F.Cu at (163.1, 69.9)
- added U5: USBLC6-2P6, Package_TO_SOT_SMD:SOT-666, F.Cu at (163.1, 73.4)
- SW3: value bootsel -> BOOT_SEL
- SW4: value SW_Push -> Programming Button
- Y1: footprint Crystal:Crystal_SMD_1210-4Pin_1.2x1.0mm -> Crystal:Crystal_SMD_Abracon_ABM8G-4Pin_3.2x2.5mm
- moved U4 96.0 mm to (179.0, 40.1)
- moved P2 86.5 mm to (170.7, 76.8)
- moved D1 83.6 mm to (179.6, 66.0)
- moved J3 69.1 mm to (148.3, 58.8)
- moved Y1 68.1 mm to (154.0, 69.1)
- moved J1 61.9 mm to (151.8, 43.1), turned to 0 degrees
- moved SW4 37.8 mm to (165.8, 37.5)
- moved C13 35.0 mm to (144.2, 71.8)
- moved C14 35.0 mm to (144.2, 73.8)
- moved C17 35.0 mm to (147.1, 71.8)
- moved C18 35.0 mm to (147.1, 73.8)
- moved C21 35.0 mm to (150.0, 71.8)
- moved C22 35.0 mm to (150.0, 73.8)
- moved C11 35.0 mm to (144.2, 67.8)
- moved C12 35.0 mm to (144.2, 69.8)
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Connections:
- net CLK renamed SD_CLK
- net CS renamed SD_CS
- net MISO renamed SD_MISO
- net MOSI renamed SD_MOSI
- D1 pad 3: +3V3 -> +5V
- J1 pad 1: +5V -> Net-(D3-A)
- J1 pad 2: D- -> DUPA-
- J1 pad 3: D+ -> DUPA+
- J2 pad 1: GPIO0 -> GPIO1
- J2 pad 2: GPIO1 -> GPIO6
- J2 pad 3: GPIO6 -> GPIO7
- J2 pad 4: GPIO7 -> GPIO8
- J2 pad 5: GPIO8 -> GPIO9
- J2 pad 6: GPIO9 -> GPIO10
- J4 pad 1: GPIO10 -> GPIO11
- J4 pad 2: GPIO11 -> GPIO12
- J4 pad 3: GPIO12 -> GPIO13
- P2 pad A4: +5V -> Net-(D2-A)
- P2 pad A6: D+ -> DUPC+
- P2 pad A7: D- -> DUPC-
- P2 pad A9: +5V -> Net-(D2-A)
- P2 pad B4: +5V -> Net-(D2-A)
- P2 pad B9: +5V -> Net-(D2-A)
- SW4 pad 1: PUSH -> GND

Commit message: pcb some few little
Parts:
- moved U3 72.8 mm to (97.5, 38.4), turned to 90 degrees
- moved J1 36.6 mm to (115.5, 38.5)
- moved P2 3.90 mm to (167.5, 79.0)
- moved U5 0.49 mm to (163.6, 73.4)
Changed lines of the file:
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@@
 	(footprint "Connector_USB:USB_A_CNCTech_1001-011-01101_Horizontal"
 		(layer "F.Cu")
-		(at 151.85 43.14)
+		(at 115.5 38.5)
 		(descr "USB type A Plug, Horizontal, http://cnctech.us/pdfs/1001-011-01101.pdf")
 		(tags "USB-A")
@@
 	(footprint "Connector_USB:USB_C_Plug_Molex_105444"
 		(layer "F.Cu")
-		(at 170.725 76.76)
+		(at 167.5 78.96)
 		(descr "Universal Serial Bus (USB) Shielded I/O Plug, Type C, Right Angle, Surface Mount, http://www.molex.com/pdm_docs/sd/1054440001_sd.pdf")
 		(tags "USB Type-C Plug Edge Mount")
@@
 	(footprint "Package_TO_SOT_SMD:SOT-666"
 		(layer "F.Cu")
-		(at 163.11 73.4)
+		(at 163.6 73.4)
 		(descr "SOT666")
 		(tags "SOT-666")
@@
 	(footprint "Package_TO_SOT_SMD:SOT-666"
 		(layer "F.Cu")
-		(at 163.11 69.945)
+		(at 97.5375 38.4 90)
 		(descr "SOT666")
 		(tags "SOT-666")
 		(property "Reference" "U3"
-			(at 0 -2 0)
+			(at 0 -2 90)
 			(layer "F.SilkS")
 			(effects
@@
 		)
 		(property "Value" "USBLC6-2P6"
-			(at 0 1.75 180)
+			(at 0 1.75 90)
 			(layer "F.Fab")
 			(effects
@@
 		)
 		(property "Datasheet" "https://www.st.com/resource/en/datasheet/usblc6-2.pdf"
-			(at 0 0 0)
+			(at 0 0 90)
 			(unlocked yes)
 			(layer "F.Fab")
@@
 		)
 		(property "Description" "Very low capacitance ESD protection diode, 2 data-line, SOT-666"
-			(at 0 0 0)
+			(at 0 0 90)
 			(unlocked yes)
 			(layer "F.Fab")
@@
 		(fp_line
 			(start -1.5 -1.1)
-			(end -1.5 1.1)
+			(end 1.5 -1.1)
 			(stroke
 				(width 0.05)
@@
 		(fp_line
 			(start -1.5 -1.1)
-			(end 1.5 -1.1)
+			(end -1.5 1.1)
 			(stroke
 				(width 0.05)
@@
 		)
 		(fp_line
-			(start -1.5 1.1)
-			(end 1.5 1.1)
+			(start 1.5 1.1)
+			(end 1.5 -1.1)
 			(stroke
 				(width 0.05)
@@
 		)
 		(fp_line
-			(start 1.5 1.1)
-			(end 1.5 -1.1)
+			(start -1.5 1.1)
+			(end 1.5 1.1)
 			(stroke
 				(width 0.05)
@@
 		)
 		(fp_line
-			(start -0.65 -0.53)
-			(end -0.65 0.85)
+			(start 0.65 -0.85)
+			(end -0.33 -0.85)
 			(stroke
 				(width 0.1)
@@
 		)
 		(fp_line
-			(start -0.65 -0.53)
+			(start 0.65 -0.85)
 			(end -0.33 -0.85)
 			(stroke
@@
 		(fp_line
 			(start 0.65 -0.85)
-			(end -0.33 -0.85)
+			(end 0.65 0.85)
 			(stroke
 				(width 0.1)
@@
 		)
 		(fp_line
-			(start 0.65 -0.85)
+			(start -0.65 -0.53)
 			(end -0.33 -0.85)
 			(stroke
@@
 		)
 		(fp_line
-			(start 0.65 -0.85)
-			(end 0.65 0.85)
+			(start -0.65 -0.53)
+			(end -0.65 0.85)
 			(stroke
 				(width 0.1)
@@
 		)
 		(fp_text user "${REFERENCE}"
-			(at 0 0 90)
+			(at 0 0 0)
 			(layer "F.Fab")
 			(effects
@@
 		)
 		(pad "1" smd roundrect
-			(at -0.85 -0.5375)
+			(at -0.85 -0.5375 90)
 			(size 0.5 0.375)
 			(layers "F.Cu" "F.Mask" "F.Paste")
@@
 		)
 		(pad "2" smd roundrect
-			(at -0.925 0)
+			(at -0.925 0 90)
 			(size 0.65 0.3)
 			(layers "F.Cu" "F.Mask" "F.Paste")
@@
 		)
 		(pad "3" smd roundrect
-			(at -0.85 0.5375)
+			(at -0.85 0.5375 90)
 			(size 0.5 0.375)
 			(layers "F.Cu" "F.Mask" "F.Paste")
@@
 		)
 		(pad "4" smd roundrect
-			(at 0.85 0.5375)
+			(at 0.85 0.5375 90)
 			(size 0.5 0.375)
 			(layers "F.Cu" "F.Mask" "F.Paste")
@@
 		)
 		(pad "5" smd roundrect
-			(at 0.925 0)
+			(at 0.925 0 90)
 			(size 0.65 0.3)
 			(layers "F.Cu" "F.Mask" "F.Paste")
@@
 		)
 		(pad "6" smd roundrect
-			(at 0.85 -0.5375)
+			(at 0.85 -0.5375 90)
 			(size 0.5 0.375)
 			(layers "F.Cu" "F.Mask" "F.Paste")

Commit message: did pcb a lil bit
Parts:
- removed BZ1: Buzzer, Buzzer_Beeper:Buzzer_CUI_CPT-9019S-SMT
- removed J5: Conn_01x03_Pin, Connector_PinSocket_2.54mm:PinSocket_1x03_P2.54mm_Vertical
- removed SW4: Programming Button, Button_Switch_THT:SW_PUSH_6mm
- added J6: Conn_01x04_Pin, Connector_PinHeader_2.54mm:PinHeader_1x04_P2.54mm_Vertical, F.Cu at (86.7, 103.5)
- D1, SW3, U1, U5: moved to B.Cu
- moved U4 97.5 mm to (90.0, 80.0)
- moved D1 90.7 mm to (90.0, 80.0), turned to 180 degrees
- moved D4 89.7 mm to (90.0, 73.8)
- moved SW3 86.0 mm to (84.2, 66.6), turned to 180 degrees
- moved P2 82.9 mm to (90.2, 109.0), turned to 180 degrees
- moved U5 82.2 mm to (88.2, 106.3), turned to -90 degrees
- moved J2 79.7 mm to (81.8, 72.7)
- moved D5 75.9 mm to (105.5, 89.6)
- moved D6 75.9 mm to (105.5, 93.2)
- moved D7 75.9 mm to (105.5, 96.7)
- moved SW2 73.7 mm to (94.3, 62.8), turned to -90 degrees
- moved J4 68.2 mm to (98.2, 72.8)
- moved J3 67.8 mm to (90.0, 93.3)
- moved U1 56.7 mm to (90.0, 91.5), turned to 180 degrees
- moved J1 26.7 mm to (90.0, 46.2), turned to 90 degrees
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Routing:
- net DUPA+: track 0.00 -> 8.39 mm
- net DUPA-: track 0.00 -> 7.64 mm
- net DUPC+: track 0.00 -> 5.11 mm, vias 0 -> 1
- net DUPC-: track 0.00 -> 4.23 mm, vias 0 -> 1
- added copper zone on F.Cu, net GND

Commit message: pcb work
Parts:
- moved U2 81.7 mm to (82.6, 107.8)
- moved J6 16.2 mm to (94.5, 117.8)
- moved J3 3.04 mm to (92.6, 94.8), turned to 90 degrees
Routing:
- net D-: track 0.00 -> 59.0 mm, vias 0 -> 1
- net D+: track 0.00 -> 58.0 mm, vias 0 -> 1
- net SD_MOSI: track 0.00 -> 24.9 mm, vias 0 -> 2
- net SD_CLK: track 0.00 -> 21.7 mm
- net SD_MISO: track 0.00 -> 17.1 mm
- added copper zone on B.Cu, net GND

Commit message: did pcb most of work done wooo
Parts:
- removed J4: Conn_01x06_Pin, Connector_PinSocket_2.54mm:PinSocket_1x06_P2.54mm_Vertical
- removed J6: Conn_01x04_Pin, Connector_PinHeader_2.54mm:PinHeader_1x04_P2.54mm_Vertical
- added G***: LOGO, kicadlogos:communism, F.Cu at (133.2, 55.2)
- added R9: 1k, Resistor_SMD:R_0402_1005Metric, F.Cu at (92.8, 87.0)
- C15: footprint Capacitor_SMD:C_0402_1005Metric -> Capacitor_SMD:C_0805_2012Metric
- C16, C8, U2: moved to B.Cu
- J2: value Conn_01x06_Pin -> Conn_02x02_Top_Bottom; footprint Connector_PinSocket_2.54mm:PinSocket_1x06_P2.54mm_Vertical -> Connector_PinHeader_1.00mm:PinHeader_2x02_P1.00mm_Vertical_SMD
- R4, R5: footprint Resistor_SMD:R_0805_2012Metric -> Capacitor_SMD:C_0402_1005Metric; moved to B.Cu
- SW3: moved to F.Cu
- moved R17 106.6 mm to (87.2, 100.5)
- moved R20 106.4 mm to (87.3, 95.0)
- moved R21 105.1 mm to (87.2, 94.0)
- moved R18 105.1 mm to (87.2, 99.5)
- moved R19 103.0 mm to (87.2, 97.2)
- moved R16 102.5 mm to (87.2, 101.5)
- moved R8 95.7 mm to (84.7, 77.2)
- moved R22 92.5 mm to (92.5, 74.8), turned to 90 degrees
- moved R7 89.1 mm to (91.5, 74.8), turned to 90 degrees
- moved R5 77.7 mm to (89.0, 106.5), turned to 90 degrees
- moved R4 77.4 mm to (91.2, 107.2)
- moved D2 76.8 mm to (83.0, 108.0)
- moved R15 72.4 mm to (81.5, 76.8), turned to 90 degrees
- moved Y1 66.8 mm to (90.0, 88.2)
- moved C17 63.4 mm to (84.0, 78.2), turned to 180 degrees
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Connections:
- C12 pad 1: XOUT -> Net-(C12-Pad1)
- J2 pad 1: GPIO1 -> GPIO23
- J2 pad 2: GPIO6 -> GPIO22
- J2 pad 3: GPIO7 -> GPIO24
- J2 pad 4: GPIO8 -> GPIO21
- Y1 pad 3: XOUT -> Net-(C12-Pad1)
Routing:
- net GPIO14: track 0.00 -> 48.8 mm, vias 0 -> 1
- net GPIO0: track 0.00 -> 47.9 mm, vias 0 -> 1
- net GPIO15: track 0.00 -> 47.6 mm, vias 0 -> 1
- net GPIO16: track 0.00 -> 32.4 mm, vias 0 -> 1
- net D-: track 59.0 -> 87.2 mm, vias 1 -> 2
- net D+: track 58.0 -> 85.6 mm, vias 1 -> 3
- net GND: track 0.00 -> 24.5 mm, vias 0 -> 17
- net SD_MOSI: track 24.9 -> 1.74 mm, vias 2 -> 0
- net Net-(R8-Pad1): track 0.00 -> 21.5 mm, vias 0 -> 2
- net SD_CLK: track 21.7 -> 1.72 mm
- net QSPI_SS: track 0.00 -> 18.2 mm, vias 0 -> 2
- net SD_MISO: track 17.1 -> 1.69 mm
- net Net-(D2-A): track 0.00 -> 14.4 mm, vias 0 -> 1
- net +3V3: track 0.00 -> 14.0 mm
- net QSPI_SD3: track 0.00 -> 11.6 mm, vias 0 -> 1
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- added copper zone on F.Cu, net +3V3
- removed copper zone on F.Cu, net GND
Other:
- board size 20 x 60 mm -> 20 x 59.5 mm

Commit message: lets end stream here eh done with qspi and sd so yea https://youtu.be/rrAUqN_xz0k
Parts:
- moved U2 1.35 mm to (82.5, 99.4)
Routing:
- net SD_CS: track 1.70 -> 26.9 mm, vias 0 -> 4
- net SD_MOSI: track 1.74 -> 26.6 mm, vias 0 -> 2
- net SD_CLK: track 1.72 -> 24.8 mm
- net SD_MISO: track 1.69 -> 21.2 mm, vias 0 -> 2
- net +3V3: track 14.0 -> 22.0 mm, vias 0 -> 2
- net GPIO0: track 47.9 -> 48.0 mm, vias 1 -> 3

Commit message: full done yayayay
Parts:
- removed D5, D6, D7: WS2812B, LED_SMD:LED_WS2812B-2020_PLCC4_2.0x2.0mm
- removed SW2: SW_DIP_x04, Button_Switch_THT:SW_DIP_SPSTx04_Slide_6.7x11.72mm_W7.62mm_P2.54mm_LowProfile
- added G***: LOGO, LOGO, F.Cu at (82.5, 84.8)
- added G***: LOGO, LOGO, F.Cu at (82.8, 65.8)
- added G***: LOGO, LOGO, F.Cu at (81.8, 101.2)
- added G***: LOGO, LOGO, F.Cu at (60.2, 85.0)
- added G***: LOGO, LOGO, B.Cu at (89.2, 90.5)
- added SW4: BOOT_SEL, Button_Switch_SMD:SW_Push_SPST_NO_Alps_SKRK, B.Cu at (92.5, 70.8)
- C12, C13, C14, D3, D4, J1, R6, R9, U3, Y1: moved to B.Cu
- SW3: footprint Button_Switch_SMD:SW_Push_1P1T_XKB_TS-1187A -> Button_Switch_SMD:SW_Push_SPST_NO_Alps_SKRK; moved to B.Cu
- moved R6 91.3 mm to (92.2, 92.6), turned to 90 degrees
- moved C19 87.3 mm to (86.5, 67.8), turned to 180 degrees
- moved C20 85.4 mm to (88.5, 67.8)
- moved D3 82.8 mm to (94.8, 95.5), turned to -90 degrees
- moved C14 74.0 mm to (95.5, 92.8), turned to 180 degrees
- moved J1 63.4 mm to (90.0, 109.7), turned to -90 degrees
- moved D2 45.1 mm to (96.7, 65.1), turned to 180 degrees
- moved P2 44.0 mm to (90.0, 64.5), turned to 0 degrees
- moved R4 41.1 mm to (88.5, 66.2), turned to 180 degrees
- moved D1 40.7 mm to (96.0, 79.2), turned to 0 degrees
- moved R5 40.0 mm to (90.7, 66.6), turned to -90 degrees
- moved U3 39.7 mm to (82.8, 98.2), turned to -90 degrees
- moved U5 38.6 mm to (95.5, 68.1), turned to 90 degrees
- moved D4 26.2 mm to (82.0, 82.0), turned to 180 degrees
- moved U2 15.5 mm to (95.0, 90.2)
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Connections:
- D4 pad 2: GPIO17 -> GPIO11
Routing:
- net +5V: track 3.90 -> 99.6 mm, vias 1 -> 10
- net +3V3: track 22.0 -> 103.6 mm, vias 2 -> 9
- net GND: track 24.5 -> 94.1 mm, vias 17 -> 30
- net GPIO14: track 48.8 -> 0.00 mm, vias 1 -> 0
- net GPIO15: track 47.6 -> 0.00 mm, vias 1 -> 0
- net GPIO16: track 32.4 -> 0.00 mm, vias 1 -> 0
- net D-: track 87.2 -> 61.4 mm
- net D+: track 85.6 -> 61.4 mm, vias 3 -> 2
- net Net-(D3-A): track 0.00 -> 12.4 mm, vias 0 -> 2
- net GPIO0: track 48.0 -> 36.6 mm
- net +1V1: track 7.43 -> 17.6 mm, vias 1 -> 3
- net Net-(R8-Pad1): track 21.5 -> 13.0 mm, vias 2 -> 3
- net SD_CS: track 26.9 -> 21.6 mm, vias 4 -> 2
- net Net-(D2-A): track 14.4 -> 19.3 mm, vias 1 -> 2
- net SD_MOSI: track 26.6 -> 21.8 mm
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Other:
- board size 20 x 59.5 mm -> 21 x 42.4 mm
- board text added: "Hackducky"
- board text added: "Souptik.me & Aarav J."
