File: hackducky.kicad_pcb (KiCad board)
At the start: 2 copper layers, 21 x 47 mm, 50 parts, among them J1 USB_A, J2 Conn_02x02_Top_Bottom, J3 Micro_SD_Card, P2 USB_C_Plug, SW3 BOOT_SEL, SW4 BOOT_SEL, U1 W25Q16JVSS, U2 AP2112K-3.3, U3 USBLC6-2P6, U4 RP2040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

Commit message: v4 done
Routing:
- net GND: track 154.9 -> 152.7 mm
- net Net-(D2-A): track 29.3 -> 28.7 mm

Commit message: silkscreen
Parts:
- removed the G*** at (93.5, 86.3) (x2)
- removed the G*** at (81.8, 101.2)
- added G*** (x2): LOGO, LOGO, F.Cu at (82.1, 93.5)
- added G*** (x2): LOGO, LOGO, B.Cu at (83.4, 93.9)
- moved D1 0.60 mm to (99.3, 80.5)
Routing:
- net +3V3: track 108.0 -> 151.4 mm, vias 17 -> 23
- net GND: track 152.7 -> 168.1 mm, vias 23 -> 33
- net Net-(D2-A): track 28.7 -> 27.0 mm
- net GP25: track 5.49 -> 6.62 mm
- added copper zone on B.Cu, net +5V
- added copper zone on F.Cu, net GND
