File: src/hackducky.kicad_pcb (KiCad board)
At the start: 2 copper layers, 21 x 47 mm, 51 parts, among them J1 USB_A, J2 Conn_02x02_Top_Bottom, J3 Micro_SD_Card, P2 USB_C_Plug, SW3 BOOT_SEL, SW4 BOOT_SEL, U1 W25Q16JVSS, U2 AP2112K-3.3, U3 USBLC6-2P6, U4 RP2040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

Commit message: update
Parts:
- moved G*** 0.53 mm to (83.3, 93.4) (x2)
- moved C7 0.50 mm to (89.0, 74.3)
- moved G*** 0.38 mm to (82.3, 93.2) (x2)
- moved R7 0.22 mm to (91.4, 74.5)
- moved R22 0.19 mm to (92.5, 74.5)
Connections:
- net Net-(U4-USB_DM) renamed DR-
- net Net-(U4-USB_DP) renamed DR+
Routing:
- net GND: track 168.1 -> 183.9 mm
- net D-: track 50.4 -> 44.2 mm
- net D+: track 50.4 -> 44.2 mm
- net Net-(D2-A): track 27.0 -> 24.8 mm, vias 3 -> 2
- net +3V3: track 151.4 -> 153.2 mm
- net DUPC+: track 18.9 -> 17.0 mm
- net DUPA+: track 15.9 -> 17.7 mm
- net Net-(P2-VCONN): track 6.02 -> 4.35 mm, vias 2 -> 1
- net DUPC-: track 18.8 -> 20.0 mm, vias 2 -> 0
- net DUPA-: track 15.9 -> 16.8 mm
- net +5V: track 72.2 -> 72.0 mm, vias 4 -> 6
- removed copper zone on F.Cu, net GND

Commit message: fix
Parts:
- moved U3 0.78 mm to (82.9, 100.5), turned to 90 degrees
- turned U5 to 180 degrees
Connections:
- U5 pad 1: D+ -> D-
- U5 pad 3: DUPC+ -> DUPC-
- U5 pad 4: DUPC- -> DUPC+
- U5 pad 6: D- -> D+
Routing:
- net D-: track 44.2 -> 3.79 mm, vias 3 -> 0
- net D+: track 44.2 -> 3.79 mm, vias 3 -> 0
- net DUPC-: track 20.0 -> 7.22 mm
- net DUPC+: track 17.0 -> 7.22 mm, vias 2 -> 0
- net DUPA+: track 17.7 -> 11.5 mm, vias 2 -> 0
- net DUPA-: track 16.8 -> 12.3 mm, vias 2 -> 0
- net +5V: track 72.0 -> 67.7 mm
- net Net-(P2-VCONN): track 4.35 -> 3.31 mm
- net Net-(D2-A): track 24.8 -> 25.5 mm
- net GND: track 183.9 -> 183.8 mm, vias 33 -> 32

Commit message: finish finally hell yeah(mostly :pf:)
Routing:
- net D+: track 3.79 -> 47.8 mm, vias 0 -> 4
- net D-: track 3.79 -> 47.8 mm, vias 0 -> 4
- net +5V: track 67.7 -> 74.1 mm
- net GND: track 183.8 -> 189.5 mm
- net +3V3: track 153.2 -> 154.5 mm
- net DUPA+: track 11.5 -> 12.2 mm
