File: src/hackducky.kicad_sch (KiCad schematic)
At the start: 46 parts, among them J1 USB_A, J2 Conn_02x02_Top_Bottom, J3 Micro_SD_Card, P2 USB_C_Plug, SW3 BOOT_SEL, SW4 BOOT_SEL, U1 W25Q16JVSS, U2 AP2112K-3.3, U3 USBLC6-2P6, U4 RP2040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

Commit message: update
Connections:
- net DR+: now reaches R7.1, U4.47 (USB_DP)
- net DR-: now reaches R22.1, U4.46 (USB_DM)
Other:
- moved on the sheet: R22, R7
Changed lines of the file:
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@@
 	(wire
 		(pts
-			(xy 283.21 85.09) (xy 288.29 85.09)
+			(xy 292.1 85.09) (xy 297.18 85.09)
 		)
 		(stroke
@@
 	(wire
 		(pts
-			(xy 270.51 87.63) (xy 275.59 87.63)
-		)
-		(stroke
-			(width 0)
-			(type default)
-		)
-	)
-	(wire
-		(pts
 			(xy 153.67 341.63) (xy 154.94 341.63)
 		)
@@
 	(wire
 		(pts
-			(xy 283.21 87.63) (xy 288.29 87.63)
+			(xy 292.1 87.63) (xy 297.18 87.63)
 		)
 		(stroke
@@
 	(wire
 		(pts
-			(xy 270.51 85.09) (xy 275.59 85.09)
-		)
-		(stroke
-			(width 0)
-			(type default)
-		)
-	)
-	(wire
-		(pts
 			(xy 195.58 50.8) (xy 208.28 50.8)
 		)
@@
 	(global_label "D+"
 		(shape input)
-		(at 288.29 85.09 0)
+		(at 297.18 85.09 0)
 		(fields_autoplaced yes)
 		(effects
@@
 		)
 		(property "Intersheetrefs" "${INTERSHEET_REFS}"
-			(at 294.1176 85.09 0)
+			(at 303.0076 85.09 0)
 			(effects
 				(font
@@
 		)
 	)
+	(global_label "DR-"
+		(shape input)
+		(at 284.48 87.63 180)
+		(fields_autoplaced yes)
+		(effects
+			(font
+				(size 1.27 1.27)
+			)
+			(justify right)
+		)
+		(property "Intersheetrefs" "${INTERSHEET_REFS}"
+			(at 277.3824 87.63 0)
+			(effects
+				(font
+					(size 1.27 1.27)
+				)
+				(justify right)
+				(hide yes)
+			)
+		)
+	)
 	(global_label "QSPI_SD3"
 		(shape input)
@@
 		)
 	)
+	(global_label "DR+"
+		(shape input)
+		(at 270.51 85.09 0)
+		(fields_autoplaced yes)
+		(effects
+			(font
+				(size 1.27 1.27)
+			)
+			(justify left)
+		)
+		(property "Intersheetrefs" "${INTERSHEET_REFS}"
+			(at 277.6076 85.09 0)
+			(effects
+				(font
+					(size 1.27 1.27)
+				)
+				(justify left)
+				(hide yes)
+			)
+		)
+	)
 	(global_label "GPIO21"
 		(shape input)
@@
 		)
 	)
+	(global_label "DR+"
+		(shape input)
+		(at 284.48 85.09 180)
+		(fields_autoplaced yes)
+		(effects
+			(font
+				(size 1.27 1.27)
+			)
+			(justify right)
+		)
+		(property "Intersheetrefs" "${INTERSHEET_REFS}"
+			(at 277.3824 85.09 0)
+			(effects
+				(font
+					(size 1.27 1.27)
+				)
+				(justify right)
+				(hide yes)
+			)
+		)
+	)
+	(global_label "DR-"
+		(shape input)
+		(at 270.51 87.63 0)
+		(fields_autoplaced yes)
+		(effects
+			(font
+				(size 1.27 1.27)
+			)
+			(justify left)
+		)
+		(property "Intersheetrefs" "${INTERSHEET_REFS}"
+			(at 277.6076 87.63 0)
+			(effects
+				(font
+					(size 1.27 1.27)
+				)
+				(justify left)
+				(hide yes)
+			)
+		)
+	)
 	(global_label "SD_CS"
 		(shape input)
@@
 	(global_label "D-"
 		(shape input)
-		(at 288.29 87.63 0)
+		(at 297.18 87.63 0)
 		(fields_autoplaced yes)
 		(effects
@@
 		)
 		(property "Intersheetrefs" "${INTERSHEET_REFS}"
-			(at 294.1176 87.63 0)
+			(at 303.0076 87.63 0)
 			(effects
 				(font
@@
 	(symbol
 		(lib_id "Device:R")
-		(at 279.4 85.09 90)
+		(at 288.29 85.09 90)
 		(unit 1)
 		(exclude_from_sim no)
@@
 		(dnp no)
 		(property "Reference" "R7"
-			(at 275.082 83.058 90)
+			(at 283.972 83.058 90)
 			(effects
 				(font
@@
 		)
 		(property "Value" "27.4"
-			(at 284.48 83.312 90)
+			(at 293.37 83.312 90)
 			(effects
 				(font
@@
 		)
 		(property "Footprint" "Resistor_SMD:R_0402_1005Metric"
-			(at 279.4 86.868 90)
+			(at 288.29 86.868 90)
 			(effects
 				(font
@@
 		)
 		(property "Datasheet" "~"
-			(at 279.4 85.09 0)
+			(at 288.29 85.09 0)
 			(effects
 				(font
@@
 		)
 		(property "Description" "Resistor"
-			(at 279.4 85.09 0)
+			(at 288.29 85.09 0)
 			(effects
 				(font
@@
 	(symbol
 		(lib_id "Device:R")
-		(at 279.4 87.63 90)
+		(at 288.29 87.63 90)
 		(unit 1)
 		(exclude_from_sim no)
@@
 		(dnp no)
 		(property "Reference" "R22"
-			(at 275.082 89.408 90)
+			(at 283.972 89.408 90)
 			(effects
 				(font
@@
 		)
 		(property "Value" "27.4"
-			(at 284.48 89.662 90)
+			(at 293.37 89.662 90)
 			(effects
 				(font
@@
 		)
 		(property "Footprint" "Resistor_SMD:R_0402_1005Metric"
-			(at 279.4 89.408 90)
+			(at 288.29 89.408 90)
 			(effects
 				(font
@@
 		)
 		(property "Datasheet" "~"
-			(at 279.4 87.63 0)
+			(at 288.29 87.63 0)
 			(effects
 				(font
@@
 		)
 		(property "Description" "Resistor"
-			(at 279.4 87.63 0)
+			(at 288.29 87.63 0)
 			(effects
 				(font

Commit message: fix
Connections:
- net D+: now also U5.6 (I/O1); no longer U5.1 (I/O1)
- net D-: now also U5.1 (I/O1); no longer U5.6 (I/O1)
- net DUPC+: now also U5.4 (I/O2); no longer U5.3 (I/O2)
- net DUPC-: now also U5.3 (I/O2); no longer U5.4 (I/O2)

Commit message: done:
Parts:
- J3: footprint Connector_Card:microSD_HC_Molex_47219-2001 -> Connector_Card:microSD_HC_Hirose_DM3AT-SF-PEJM5
Changed lines of the file:
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@@
 			)
 		)
-		(property "Footprint" "Connector_Card:microSD_HC_Molex_47219-2001"
+		(property "Footprint" "Connector_Card:microSD_HC_Hirose_DM3AT-SF-PEJM5"
 			(at 102.87 265.43 0)
 			(effects

Commit message: 2nd v
Parts:
- removed D2, D3: MBR1020VL, Diode_SMD:D_SOD-123F, symbol Diode:MBR1020VL
- removed R6: 5.1K, Resistor_SMD:R_0805_2012Metric, symbol Device:R
- removed U2: AP2112K-3.3, Package_TO_SOT_SMD:SOT-23-5, symbol Regulator_Linear:AP2112K-3.3
- removed U3, U5: USBLC6-2P6, Package_TO_SOT_SMD:SOT-666, symbol Power_Protection:USBLC6-2P6
- added C23: 22uF, Capacitor_SMD:C_0402_1005Metric, symbol Device:C
- added D5, D6: LED, LED_SMD:LED_0603_1608Metric, symbol Device:LED
- added FB1, FB2: 120ohm.100Mhz, Inductor_SMD:L_0805_2012Metric, symbol Device:FerriteBead
- added R1, R2: R, Resistor_SMD:R_0402_1005Metric, symbol Device:R
- added TP1, TP10, TP11, TP12, TP2, TP3, TP4, TP5, TP6, TP7, TP8, TP9: TestPoint, TestPoint:TestPoint_Pad_D1.0mm, symbol Connector:TestPoint
- added U2: AMS1117-3.3, Package_TO_SOT_SMD:SOT-223-3_TabPin2, symbol Regulator_Linear:AMS1117-3.3
- C14: value 1uF -> 22uF
- C15: value 1uF -> 22uF; footprint Capacitor_SMD:C_0805_2012Metric -> Capacitor_SMD:C_0402_1005Metric
- C22: value 100n -> 100nF
- R15: footprint Resistor_SMD:R_0805_2012Metric_Pad1.20x1.40mm_HandSolder -> Resistor_SMD:R_0402_1005Metric
Connections:
- net DUPA+ is gone; now on net D+: J1.3 (D+)
- net DUPA- is gone; now on net D-: J1.2 (D-)
- net DUPC+ is gone; now on net D+: P2.A6 (D+)
- net DUPC- is gone; now on net D-: P2.A7 (D-)
- net +3V3: now also D5.2 (A), U2.2 (VO)
- net +5V: now also C23.1, D6.2 (A), FB1.2, FB2.2, TP10.1, TP11.1, TP12.1, TP7.1, TP8.1, TP9.1, U2.3 (VI)
- net GND: now also C23.2, R1.2, R2.2, TP1.1, TP2.1, TP3.1, TP4.1, TP5.1, TP6.1, U2.1 (GND)
- net VBUS: now reaches J1.1 (VBUS)
- net VBUS: now also P2.A4 (VBUS), P2.A9 (VBUS), P2.B4 (VBUS), P2.B9 (VBUS), FB1.1, FB2.1
- new net: D5.1 (K), R1.1
- new net: D6.1 (K), R2.1

Commit message: 2nd v
Parts:
- added C24, C25: 100nF, Capacitor_SMD:C_0402_1005Metric, symbol Device:C
Connections:
- net +1V1: now also TP1.1, TP2.1, C25.2
- net +3V3: now also TP10.1, TP7.1, C24.2
- net +5V: no longer TP10.1, TP7.1
- net GND: now also C24.1, C25.1; no longer TP1.1, TP2.1
