File: src/hackducky.kicad_sch (KiCad schematic)
At the start: 62 parts, among them J1 USB_A, J2 Conn_02x02_Top_Bottom, J3 Micro_SD_Card, P2 USB_C_Plug, SW3 BOOT_SEL, SW4 BOOT_SEL, U1 W25Q16JVSS, U2 AMS1117-3.3, U4 RP2040, Y1 Crystal_GND24

Commit message: 2nd v
Other:
- moved on the sheet: C14, C15, C23, D5, D6, R1, R2, U2

Commit message: f
Parts:
- removed R5: 5.1K, Capacitor_SMD:C_0402_1005Metric, symbol Device:R
- added U5, U6: SRV05-4, Package_TO_SOT_SMD:SOT-23-6, symbol Power_Protection:SRV05-4
Connections:
- net +3V3: now also U5.5 (VP), U6.5 (VP)
- net D+: now also U5.1 (IO1), U6.1 (IO1)
- net D-: now also U5.3 (IO2), U6.3 (IO2)
- net GND: now also U5.2 (VN), U6.2 (VN)

Commit message: f
Parts:
- P2: footprint Connector_USB:USB_C_Plug_Molex_105444 -> RASPBERRY_PI_PICO:USB-C-SMD_U261-121N-4BS2S
Changed lines of the file:
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@@
 			)
 		)
-		(property "Footprint" "Connector_USB:USB_C_Plug_Molex_105444"
+		(property "Footprint" "RASPBERRY_PI_PICO:USB-C-SMD_U261-121N-4BS2S"
 			(at 36.83 95.25 0)
 			(effects

Commit message: first commit
Parts:
- removed U1: W25Q16JVSS, Package_SO:SOIC-8_5.3x5.3mm_P1.27mm, symbol Memory_Flash:W25Q16JVSS
- added C1: 1uF, Capacitor_SMD:C_0402_1005Metric, symbol Device:C
- added J4: Conn_01x03_Pin, Connector_PinHeader_1.27mm:PinHeader_1x03_P1.27mm_Vertical, symbol Connector:Conn_01x03_Pin
- added J6: Conn_01x04_Pin, Connector_PinHeader_1.00mm:PinHeader_1x04_P1.00mm_Vertical, symbol Connector:Conn_01x04_Pin
- added JP1: Jumper_2_Open, Jumper:SolderJumper-2_P1.3mm_Open_RoundedPad1.0x1.5mm, symbol Jumper:Jumper_2_Open
- added U3: W25Q128JVS, Package_SO:SOIC-8_5.3x5.3mm_P1.27mm, symbol Memory_Flash:W25Q128JVS
- SW4: value BOOT_SEL -> GP0
Connections:
- net +3V3: now also C1.1, J6.1 (Pin_1), JP1.2 (B), U3.8 (VCC); no longer R15.1
- net GND: now also C1.2, J6.2 (Pin_2), U3.4 (GND)
- net GPIO6: no longer U4.8 (GPIO6)
- net GPIO7: no longer U4.9 (GPIO7)
- net QSPI_SCLK: now also U3.6 (CLK)
- net QSPI_SD0: now also U3.5 (DI/IO_{0})
- net QSPI_SD1: now also U3.2 (DO/IO_{1})
- net QSPI_SD2: now also U3.3 (~{WP}/IO_{2})
- net QSPI_SD3: now also U3.7 (~{HOLD}/~{RESET}/IO_{3})
- net QSPI_SS: now also U3.1 (~{CS})
- net RUN: now also J4.1 (Pin_1)
- net SWCLK: now also J4.3 (Pin_3)
- net SWD: now also J4.2 (Pin_2)
- new net: JP1.1 (A), R15.1
- new net I+: J6.4 (Pin_4), U4.8 (GPIO6)
- new net I-: J6.3 (Pin_3), U4.9 (GPIO7)
- no-connect marks 23 -> 21
Other:
- moved on the sheet: U5, U6

Commit message: I am done
Parts:
- removed D1, D4: WS2812B, LED_SMD:LED_SK6812_EC15_1.5x1.5mm, symbol LED:SK6812
- added D2, D3: LED, LED_SMD:LED_0402_1005Metric, symbol Device:LED
- added R3, R5: 220, Resistor_SMD:R_0402_1005Metric, symbol Device:R
- C14, C15, C23: footprint Capacitor_SMD:C_0402_1005Metric -> Capacitor_SMD:C_0603_1608Metric
Connections:
- net GND: now also R3.2, R5.2
- net GP25: now also D3.2 (A)
- net GPIO11: now also D2.2 (A)
- new net: D2.1 (K), R3.1
- new net: D3.1 (K), R5.1
- no-connect marks 21 -> 19

Commit message: final done with calip
Parts:
- added D1, D4: LED, LED_SMD:LED_0402_1005Metric, symbol Device:LED
- added R10, R6: 220, Resistor_SMD:R_0402_1005Metric, symbol Device:R
Connections:
- net GND: now also R10.2, R6.2
- net GPIO26_ADC0: now also D1.2 (A)
- net GPIO26_ADC1: no longer U4.39 (GPIO27_ADC1)
- net GPIO26_ADC3: no longer U4.41 (GPIO29_ADC3)
- new net: D1.1 (K), R6.1
- new net: D4.1 (K), R10.1
- new net GPIO27_ADC1: D4.2 (A), U4.39 (GPIO27_ADC1)
- new net GPIO29_ADC3: U4.41 (GPIO29_ADC3)
