File: Pcb/hackducky.kicad_sch (KiCad schematic)
At the start: 73 parts, among them J1 USB_A, J2 Conn_02x02_Top_Bottom, J3 Micro_SD_Card, J4 Conn_01x03_Pin, J6 Conn_01x04_Pin, P2 USB_C_Plug, SW3 BOOT_SEL, SW4 GP0, U2 AMS1117-3.3, U3 W25Q128JVS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

Commit message: POLISH
Connections:
- net DI+ is gone; now on net D+: J1.3 (D+)
- net DI- is gone; now on net D-: J1.2 (D-)
- net GND: now also R1.2, R2.2; no longer R1.1, R2.1
- net at D5.1 (K): now also R1.1; no longer R1.2
- net at D6.1 (K): now also R2.1; no longer R2.2
- no-connect marks 10 -> 19
Other:
- note added: "keep caps near (to myself)(souptik)"
- note added: "never gonna give u ip"
- note added: "sd spi"
- note removed: "Crystal"
- note removed: "ESD Protection"
- note removed: "FLASH"
- note removed: "GPIO BREAKOUT"
- note removed: "Onboard Led and Buttons"
- note removed: "Power Section and leds"
- note removed: "RP2040 with decoupling capacitors"
- note removed: "SD Card"
- note removed: "Test Pads"
- note removed: "USB C & A MALE"
- note removed: "keep caps near"
- company: Hack Industries -> (none)
- title: Hackducky -> HACKDUCKY BY SOUPTIK 
- moved on the sheet: C1, C10, C11, C12, C13, C14, C15, C16, C17, C18, C19, C20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
